File: PowerDistribution/KiCad/MegaShield.kicad_pcb (KiCad board)
At the start: 2 copper layers, 99.4 x 53 mm, 40 parts, among them IC1 L298SO, IC2 L298SO, J1 DCJ0202, J2 M03LOCK, J3 M03LOCK, J4 M03LOCK, J5 M03LOCK, J6 M03LOCK, J7 M03LOCK

Commit message: Revert "added outline gerber file"
This reverts commit 9dad513005639610b03bd811ee575d7d2b60979b.
Routing:
- added copper zone on F.Cu, net /12V
- added copper zone on B.Cu, net /GND
